Commit message: Lidar on the bottom + altitude relay

File: urdf_drone/parrot.gazebo.xacro (robot description, xacro)
@@ -171,3 +171,34 @@
     </sensor>
   </gazebo>
+  <gazebo reference="lidar_scan">
+    <material>Gazebo/FlatBlack</material>
+    <sensor type="gpu_lidar" name="lidardown">
+      <pose relative_to='lidar_scan'>0 0 0 0 0 0</pose>
+      <visualize>$(arg laser_visual)</visualize>
+      <topic>model/parrot/downscan</topic>
+      <update_rate>3</update_rate>
+      <gz_frame_id>lidar_scan</gz_frame_id>
+      <ray>
+        <scan>
+          <horizontal>
+            <samples>360</samples>
+            <resolution>1</resolution>
+            <min_angle>-1.57</min_angle>
+            <max_angle>1.57</max_angle>
+          </horizontal>
+        </scan>
+        <range>
+          <min>0.01</min>
+          <max>10</max>
+          <resolution>0.015</resolution>
+        </range>
+        <noise>
+          <type>gaussian</type>
+          <mean>0.0</mean>
+          <stddev>0.01</stddev>
+        </noise>
+      </ray>
+      <always_on>true</always_on>
+    </sensor>
+  </gazebo>
 </robot>

File: urdf_drone/parrot.urdf.xacro (robot description, xacro)
@@ -79,6 +79,27 @@
     </inertial>
   </link>
+  <joint name="lidar_joint" type="fixed">
+    <parent link="base_link"/>
+    <child link="lidar_scan"/>
+    <origin xyz="0 0 -0.035" rpy="0 0 1.57"/>
+  </joint>
+  <link name="lidar_scan">
+    <visual>
+      <origin xyz="0 0 0" rpy="0 0 0"/>
+      <geometry>
+        <cylinder length="0.01" radius="0.03"/>
+      </geometry>
+      <material name="dark"/>
+    </visual>
+    <inertial>
+      <mass value="0" />
+      <origin xyz="0 0 0" />
+      <inertia ixx="0.001" ixy="0.0" ixz="0.0"
+               iyy="0.001" iyz="0.0"
+               izz="0.001" />
+    </inertial>
+  </link>
   <joint name="camera_joint" type="fixed">
-    <origin xyz="0.25 0.0 0.25" rpy="0 0.785398 0"/> <!-- 0.5 0.0 0.9 -->
+    <origin xyz="0.25 0.0 0.25" rpy="0 0.785 0"/> <!-- 0.5 0.0 0.9 -->
     <parent link="base_link"/>
     <child link="camera_link"/>
@@ -113,5 +134,5 @@
   <link name="camera_rgb_optical_frame"/>
   <joint name="camera_depth_joint" type="fixed">
-    <origin xyz="${r200_cam_rgb_px} ${r200_cam_rgb_py + r200_cam_depth_offset} ${r200_cam_rgb_pz}" rpy="0 0 0"/>
+    <origin xyz="${r200_cam_rgb_px} ${r200_cam_rgb_py + r200_cam_depth_offset} ${r200_cam_rgb_pz}" rpy="0 1.57 0"/>
     <parent link="camera_link"/>
     <child link="camera_depth_frame"/>

Commit message: merging of flight control

File: urdf_drone/parrot.gazebo.xacro (robot description, xacro)
@@ -110,5 +110,5 @@
     <material>Gazebo/FlatBlack</material>
     <sensor type="gpu_lidar" name="lidar">
-      <pose relative_to='base_scan'>0 0 0 0 0 0</pose>
+      <pose relative_to='base_scan'>0 0 0 -1.5708 0 0</pose>
       <visualize>$(arg laser_visual)</visualize>
       <topic>model/parrot/scan</topic>

File: urdf_drone/parrot.urdf.xacro (robot description, xacro)
@@ -82,5 +82,5 @@
     <parent link="base_link"/>
     <child link="lidar_scan"/>
-    <origin xyz="0 0 -0.035" rpy="0 1.57 1.57"/>
+    <origin xyz="0 0 -0.035" rpy="0 0 0"/>
   </joint>
   <link name="lidar_scan">

Commit message: Fixing LIDAR

File: urdf_drone/parrot.gazebo.xacro (robot description, xacro)
@@ -110,5 +110,5 @@
     <material>Gazebo/FlatBlack</material>
     <sensor type="gpu_lidar" name="lidar">
-      <pose relative_to='base_scan'>0 0 0 -1.5708 0 0</pose>
+      <pose relative_to='base_scan'>0 0 0 0 0 0</pose>
       <visualize>$(arg laser_visual)</visualize>
       <topic>model/parrot/scan</topic>

File: urdf_drone/parrot.urdf.xacro (robot description, xacro)
@@ -82,5 +82,5 @@
     <parent link="base_link"/>
     <child link="lidar_scan"/>
-    <origin xyz="0 0 -0.035" rpy="0 0 0"/>
+    <origin xyz="0 0 -0.035" rpy="0 1.57 1.57"/>
   </joint>
   <link name="lidar_scan">

Commit message: cleanup

File: urdf_drone/parrot.gazebo.xacro (robot description, xacro)
@@ -171,3 +171,34 @@
     </sensor>
   </gazebo>
+  <gazebo reference="lidar_scan">
+    <material>Gazebo/FlatBlack</material>
+    <sensor type="gpu_lidar" name="lidardown">
+      <pose relative_to='lidar_scan'>0 0 0 0 0 0</pose>
+      <visualize>$(arg laser_visual)</visualize>
+      <topic>model/parrot/downscan</topic>
+      <update_rate>3</update_rate>
+      <gz_frame_id>lidar_scan</gz_frame_id>
+      <ray>
+        <scan>
+          <horizontal>
+            <samples>360</samples>
+            <resolution>1</resolution>
+            <min_angle>-1.57</min_angle>
+            <max_angle>1.57</max_angle>
+          </horizontal>
+        </scan>
+        <range>
+          <min>0.01</min>
+          <max>10</max>
+          <resolution>0.015</resolution>
+        </range>
+        <noise>
+          <type>gaussian</type>
+          <mean>0.0</mean>
+          <stddev>0.01</stddev>
+        </noise>
+      </ray>
+      <always_on>true</always_on>
+    </sensor>
+  </gazebo>
 </robot>

File: urdf_drone/parrot.urdf.xacro (robot description, xacro)
@@ -79,6 +79,27 @@
     </inertial>
   </link>
+  <joint name="lidar_joint" type="fixed">
+    <parent link="base_link"/>
+    <child link="lidar_scan"/>
+    <origin xyz="0 0 0" rpy="0 0 0"/>
+  </joint>
+  <link name="lidar_scan">
+    <visual>
+      <origin xyz="0 0 0" rpy="0 0 0"/>
+      <geometry>
+        <cylinder length="0.01" radius="0.03"/>
+      </geometry>
+      <material name="dark"/>
+    </visual>
+    <inertial>
+      <mass value="0" />
+      <origin xyz="0 0 0" />
+      <inertia ixx="0.001" ixy="0.0" ixz="0.0"
+               iyy="0.001" iyz="0.0"
+               izz="0.001" />
+    </inertial>
+  </link>
   <joint name="camera_joint" type="fixed">
-    <origin xyz="0.25 0.0 0.25" rpy="0 0.785398 0"/> <!-- 0.5 0.0 0.9 -->
+    <origin xyz="0.25 0.0 0.25" rpy="0 0.785 0"/> <!-- 0.5 0.0 0.9 -->
     <parent link="base_link"/>
     <child link="camera_link"/>
@@ -113,5 +134,5 @@
   <link name="camera_rgb_optical_frame"/>
   <joint name="camera_depth_joint" type="fixed">
-    <origin xyz="${r200_cam_rgb_px} ${r200_cam_rgb_py + r200_cam_depth_offset} ${r200_cam_rgb_pz}" rpy="0 0 0"/>
+    <origin xyz="${r200_cam_rgb_px} ${r200_cam_rgb_py + r200_cam_depth_offset} ${r200_cam_rgb_pz}" rpy="0 1.57 0"/>
     <parent link="camera_link"/>
     <child link="camera_depth_frame"/>
