Commit message: GUI

File: urdf_drone/parrot.urdf.xacro (robot description, xacro)
@@ -1,6 +1,6 @@
 <?xml version="1.0" ?>
 <robot name="parrot" xmlns:xacro="http://ros.org/wiki/xacro">
-  <xacro:include filename="$(find 41068_ignition_bringup)/urdf_drone/common_properties.urdf.xacro"/>
-  <xacro:include filename="$(find 41068_ignition_bringup)/urdf_drone/parrot.gazebo.xacro"/>
+  <xacro:include filename="$(find trailblazer)/urdf_drone/common_properties.urdf.xacro"/>
+  <xacro:include filename="$(find trailblazer)/urdf_drone/parrot.gazebo.xacro"/>
   <xacro:property name="r200_cam_rgb_px" value="0.005"/>
   <xacro:property name="r200_cam_rgb_py" value="0.018"/>
@@ -24,5 +24,5 @@
     <visual name="hull">
       <geometry>
-        <mesh filename="file://$(find 41068_ignition_bringup)/urdf_drone/meshes/hull.dae"/>
+        <mesh filename="file://$(find trailblazer)/urdf_drone/meshes/hull.dae"/>
       </geometry>
     </visual>
@@ -30,5 +30,5 @@
       <origin xyz="-0.09035 -0.11423 -0.00501" rpy="0 0 0"/>
       <geometry>
-        <mesh filename="file://$(find 41068_ignition_bringup)/urdf_drone/meshes/propeller_rr.dae"/>
+        <mesh filename="file://$(find trailblazer)/urdf_drone/meshes/propeller_rr.dae"/>
       </geometry>
     </visual>
@@ -36,5 +36,5 @@
       <origin xyz="0.09035 0.11452 -0.00501" rpy="0 0 0"/>
       <geometry>
-        <mesh filename="file://$(find 41068_ignition_bringup)/urdf_drone/meshes/propeller_rl.dae"/>
+        <mesh filename="file://$(find trailblazer)/urdf_drone/meshes/propeller_rl.dae"/>
       </geometry>
     </visual>
@@ -42,5 +42,5 @@
       <origin xyz="0.08456 -0.11435 -0.00501" rpy="0 0 0"/>
       <geometry>
-        <mesh filename="file://$(find 41068_ignition_bringup)/urdf_drone/meshes/propeller_fr.dae"/>
+        <mesh filename="file://$(find trailblazer)/urdf_drone/meshes/propeller_fr.dae"/>
       </geometry>
     </visual>
@@ -48,5 +48,5 @@
       <origin xyz="0.08456 0.11463 -0.00501" rpy="0 0 0"/>
       <geometry>
-        <mesh filename="file://$(find 41068_ignition_bringup)/urdf_drone/meshes/propeller_fl.dae"/>
+        <mesh filename="file://$(find trailblazer)/urdf_drone/meshes/propeller_fl.dae"/>
       </geometry>
     </visual>

Commit message: Starting flight control

File: urdf_drone/parrot.urdf.xacro (robot description, xacro)
@@ -16,10 +16,10 @@
                izz="3.328e-3" />
     </inertial>
-<!--     <collision name="collision">
+    <collision name="collision">
       <origin xyz="-0.00424 0.00014 -0.00595" rpy="0 0 0"/>
       <geometry>
         <box size="0.5 0.5 0.2"/>
       </geometry>
-    </collision> -->
+    </collision>
     <visual name="hull">
       <geometry>

Commit message: Fixing Down Lidar

File: urdf_drone/parrot.urdf.xacro (robot description, xacro)
@@ -82,5 +82,5 @@
     <parent link="base_link"/>
     <child link="lidar_scan"/>
-    <origin xyz="0 0 -0.035" rpy="0 0 1.57"/>
+    <origin xyz="0 0 -0.035" rpy="0 1.57 1.57"/>
   </joint>
   <link name="lidar_scan">

Commit message: Height adjustment

File: urdf_drone/parrot.urdf.xacro (robot description, xacro)
@@ -82,5 +82,5 @@
     <parent link="base_link"/>
     <child link="lidar_scan"/>
-    <origin xyz="0 0 0" rpy="0 0 0"/>
+    <origin xyz="0 0 -0.035" rpy="0 1.57 1.57"/>
   </joint>
   <link name="lidar_scan">
